Commit message: Fix arms

File: 2020/urdf/darwin.urdf (robot description, URDF)
Before this commit: robot darwin, 93 links, 92 joints
Links:
- removed link l_biceps_anchor_link
- removed link l_biceps_axis_link
- removed link l_biceps_spo_link
- removed link l_elbow_axis_link
- removed link l_elbow_link
- removed link l_elbow_spo_link
- removed link l_hand_back_link
- removed link l_hand_base_link
- removed link l_hand_fingers_ext1_link
- removed link l_hand_fingers_ext2_link
- removed link l_hand_fingers_int1_link
- removed link l_hand_fingers_int2_link
- removed link l_hand_palm_anchor1_link
- removed link l_hand_palm_anchor2_link
- removed link l_hand_palm_link
- removed link l_hand_thumb_link
- removed link l_hand_wrist1_link
- removed link l_hand_wrist2_link
- removed link l_lower_arm_link
- removed link l_upper_arm_link
- removed link l_wrist_anchor_link
- removed link r_biceps_anchor_link
- removed link r_biceps_axis_link
- removed link r_biceps_spo_link
- removed link r_elbow_axis_link
- removed link r_elbow_link
- removed link r_elbow_spo_link
- removed link r_hand_back_link
- removed link r_hand_base_link
- removed link r_hand_fingers_ext1_link
- removed link r_hand_fingers_ext2_link
- removed link r_hand_fingers_int1_link
- removed link r_hand_fingers_int2_link
- removed link r_hand_palm_anchor1_link
- removed link r_hand_palm_anchor2_link
- removed link r_hand_palm_link
- removed link r_hand_thumb_link
- removed link r_hand_wrist1_link
- removed link r_hand_wrist2_link
- removed link r_lower_arm_link
- removed link r_upper_arm_link
- removed link r_wrist_anchor_link
- added link l_hand_link, mass 0.02; collision mesh filename=meshes/l_hand.dae scale=1 1 1; visual mesh filename=meshes/l_hand.dae scale=1 1 1
- added link r_hand_link, mass 0.02; collision mesh filename=meshes/r_hand.dae scale=1 1 1; visual mesh filename=meshes/r_hand.dae scale=1 1 1
- link l_biceps_link: geometry collision mesh filename=meshes/l_biceps.dae scale=1 1 1; visual mesh filename=meshes/l_biceps.dae scale=1 1 1
- link l_shoulder_link: mass 0.0001 -> 0.005; geometry collision mesh filename=meshes/l_shoulder.dae scale=1 1 1; visual mesh filename=meshes/l_shoulder.dae scale=1 1 1
- link r_biceps_link: geometry collision mesh filename=meshes/r_biceps.dae scale=1 1 1; visual mesh filename=meshes/r_biceps.dae scale=1 1 1
- link r_shoulder_link: mass 0.0001 -> 0.005; geometry collision mesh filename=meshes/r_shoulder.dae scale=1 1 1; visual mesh filename=meshes/r_shoulder.dae scale=1 1 1
Joints:
- removed joint l_biceps_anchor_joint
- removed joint l_biceps_axis_joint
- removed joint l_biceps_spo_joint
- removed joint l_elbow_axis_joint
- removed joint l_elbow_spo_joint
- removed joint l_hand_back_joint
- removed joint l_hand_base_joint
- removed joint l_hand_fingers_ext1_joint
- removed joint l_hand_fingers_ext2_joint
- removed joint l_hand_fingers_int1_joint
- removed joint l_hand_fingers_int2_joint
- removed joint l_hand_palm_anchor1_joint
- removed joint l_hand_palm_anchor2_joint
- removed joint l_hand_palm_joint
- removed joint l_hand_thumb_joint
- removed joint l_hand_wrist1_joint
- removed joint l_hand_wrist2_joint
- removed joint l_lower_arm_joint
- removed joint l_upper_arm_joint
- removed joint l_wrist_anchor_joint
- removed joint r_biceps_anchor_joint
- removed joint r_biceps_axis_joint
- removed joint r_biceps_spo_joint
- removed joint r_elbow_axis_joint
- removed joint r_elbow_spo_joint
- removed joint r_hand_back_joint
- removed joint r_hand_base_joint
- removed joint r_hand_fingers_ext1_joint
- removed joint r_hand_fingers_ext2_joint
- removed joint r_hand_fingers_int1_joint
- removed joint r_hand_fingers_int2_joint
- removed joint r_hand_palm_anchor1_joint
- removed joint r_hand_palm_anchor2_joint
- removed joint r_hand_palm_joint
- removed joint r_hand_thumb_joint
- removed joint r_hand_wrist1_joint
- removed joint r_hand_wrist2_joint
- removed joint r_lower_arm_joint
- removed joint r_upper_arm_joint
- removed joint r_wrist_anchor_joint
- joint l_biceps_joint: parent l_biceps_axis_link -> l_shoulder_link
- joint l_elbow_joint: child l_elbow_link -> l_hand_link; origin xyz=0 0 0 rpy=0 0 -2.61799387799 -> xyz=0 0 -0.044 rpy=0 0 -2.61799387799; parent l_elbow_axis_link -> l_biceps_link
- joint l_shoulder_joint: origin xyz=0 0 0 rpy=0 0 -2.61799387799 -> xyz=-0.014 0.057 0.03 rpy=0 0 -2.61799387799
- joint r_biceps_joint: parent r_biceps_axis_link -> r_shoulder_link
- joint r_elbow_joint: child r_elbow_link -> r_hand_link; origin xyz=0 0 0 rpy=0 0 -2.61799387799 -> xyz=0 0 -0.044 rpy=0 0 -2.61799387799; parent r_elbow_axis_link -> r_biceps_link
- joint r_shoulder_joint: origin xyz=0 0 0 rpy=0 0 -2.61799387799 -> xyz=-0.014 -0.057 0.03 rpy=0 0 -2.61799387799

Commit message: Simplify robot model.  Looks OK.

File: 2020/urdf/darwin.urdf (robot description, URDF)
Before this commit: robot darwin, 53 links, 52 joints
Links:
- removed link l_achiles_link
- removed link l_ankle_axis_link
- removed link l_ankle_spo_link
- removed link l_foot_anchor_link
- removed link l_foot_axis_link
- removed link l_forefoot_link
- removed link l_groin_link
- removed link l_hip_anchor_link
- removed link l_knee_link
- removed link l_knee_servo_link
- removed link l_knee_spo_link
- removed link l_lower_leg_link
- removed link l_sole_link
- removed link l_thigh_anchor_link
- removed link l_thigh_servo_link
- removed link l_thigh_spo_link
- removed link l_thigh_top_link
- removed link l_upper_leg_link
- removed link r_achiles_link
- removed link r_ankle_axis_link
- removed link r_ankle_spo_link
- removed link r_foot_anchor_link
- removed link r_foot_axis_link
- removed link r_forefoot_link
- removed link r_groin_link
- removed link r_hip_anchor_link
- removed link r_knee_link
- removed link r_knee_servo_link
- removed link r_knee_spo_link
- removed link r_lower_leg_link
- removed link r_sole_link
- removed link r_thigh_anchor_link
- removed link r_thigh_servo_link
- removed link r_thigh_spo_link
- removed link r_thigh_top_link
- removed link r_upper_leg_link
- added link l_lowerleg_link, mass 0.001; collision mesh filename=meshes/l_lowerleg.dae scale=1 1 1; visual mesh filename=meshes/l_lowerleg.dae scale=1 1 1
- added link r_lowerleg_link, mass 0.001; collision mesh filename=meshes/r_lowerleg.dae scale=1 1 1; visual mesh filename=meshes/r_lowerleg.dae scale=1 1 1
- link l_ankle_link: geometry collision mesh filename=meshes/l_ankle.dae scale=1 1 1; visual mesh filename=meshes/l_ankle.dae scale=1 1 1
- link l_foot_link: mass 0.02 -> 0.016; geometry collision mesh filename=meshes/l_foot.dae scale=1 1 1; visual mesh filename=meshes/l_foot.dae scale=1 1 1
- link l_hip_link: mass 0.0001 -> 0.001; geometry collision mesh filename=meshes/l_hip.dae scale=1 1 1; visual mesh filename=meshes/l_hip.dae scale=1 1 1
- link l_thigh_link: mass 0.0001 -> 0.001; geometry collision mesh filename=meshes/l_thigh.dae scale=1 1 1; visual mesh filename=meshes/l_thigh.dae scale=1 1 1
- link r_ankle_link: geometry collision mesh filename=meshes/r_ankle.dae scale=1 1 1; visual mesh filename=meshes/r_ankle.dae scale=1 1 1
- link r_foot_link: mass 0.02 -> 0.016; geometry collision mesh filename=meshes/r_foot.dae scale=1 1 1; visual mesh filename=meshes/r_foot.dae scale=1 1 1
- link r_hip_link: mass 0.0001 -> 0.001; geometry collision mesh filename=meshes/r_hip.dae scale=1 1 1; visual mesh filename=meshes/r_hip.dae scale=1 1 1
- link r_thigh_link: mass 0.0001 -> 0.001; geometry collision mesh filename=meshes/r_thigh.dae scale=1 1 1; visual mesh filename=meshes/r_thigh.dae scale=1 1 1
Joints:
- removed joint l_achiles_joint
- removed joint l_ankle_axis_joint
- removed joint l_ankle_spo_joint
- removed joint l_foot_anchor_joint
- removed joint l_foot_axis_joint
- removed joint l_forefoot_joint
- removed joint l_groin_joint
- removed joint l_hip_anchor_joint
- removed joint l_knee_servo_joint
- removed joint l_knee_spo_joint
- removed joint l_lower_leg_joint
- removed joint l_sole_joint
- removed joint l_thigh_anchor_joint
- removed joint l_thigh_servo_joint
- removed joint l_thigh_spo_joint
- removed joint l_thigh_top_joint
- removed joint l_upper_leg_joint
- removed joint r_achiles_joint
- removed joint r_ankle_axis_joint
- removed joint r_ankle_spo_joint
- removed joint r_foot_anchor_joint
- removed joint r_foot_axis_joint
- removed joint r_forefoot_joint
- removed joint r_groin_joint
- removed joint r_hip_anchor_joint
- removed joint r_knee_servo_joint
- removed joint r_knee_spo_joint
- removed joint r_lower_leg_joint
- removed joint r_sole_joint
- removed joint r_thigh_anchor_joint
- removed joint r_thigh_servo_joint
- removed joint r_thigh_spo_joint
- removed joint r_thigh_top_joint
- removed joint r_upper_leg_joint
- joint l_ankle_joint: origin xyz=0 0 0 rpy=0 0 -2.61799387799 -> xyz=0 0 -0.042 rpy=0 0 -2.61799387799; parent l_ankle_axis_link -> l_lowerleg_link
- joint l_biceps_joint: axis 0 0 1 -> 1 0 0; origin xyz=0 0 0 rpy=0 0 -2.61799387799 -> xyz=0 0 0 rpy=-2.61799387799 0 0
- joint l_foot_joint: origin xyz=0 0 0 rpy=0 0 -2.61799387799 -> xyz=-0.033 0 0 rpy=0 0 -2.61799387799; parent l_foot_axis_link -> l_ankle_link
- joint l_hip_joint: origin xyz=0 0 0 rpy=0 0 -2.61799387799 -> xyz=-0.024 0.024 -0.03 rpy=0 0 -2.61799387799
- joint l_knee_joint: child l_knee_link -> l_lowerleg_link; origin xyz=0 0 0 rpy=0 0 -2.61799387799 -> xyz=0 0 -0.046 rpy=0 0 -2.61799387799; parent l_knee_servo_link -> l_thigh_link
- joint l_thigh_joint: origin xyz=0 0 0 rpy=0 0 -2.61799387799 -> xyz=0.02 0 -0.006 rpy=0 0 -2.61799387799; parent l_thigh_servo_link -> l_hip_link
- joint r_ankle_joint: origin xyz=0 0 0 rpy=0 0 -2.61799387799 -> xyz=0 0 -0.042 rpy=0 0 -2.61799387799; parent r_ankle_axis_link -> r_lowerleg_link
- joint r_biceps_joint: axis 0 0 1 -> 1 0 0; origin xyz=0 0 0 rpy=0 0 -2.61799387799 -> xyz=0 0 0 rpy=-2.61799387799 0 0
- joint r_foot_joint: origin xyz=0 0 0 rpy=0 0 -2.61799387799 -> xyz=-0.033 0 0 rpy=0 0 -2.61799387799; parent r_foot_axis_link -> r_ankle_link
- joint r_hip_joint: origin xyz=0 0 0 rpy=0 0 -2.61799387799 -> xyz=-0.024 -0.024 -0.03 rpy=0 0 -2.61799387799
- joint r_knee_joint: child r_knee_link -> r_lowerleg_link; origin xyz=0 0 0 rpy=0 0 -2.61799387799 -> xyz=0 0 -0.046 rpy=0 0 -2.61799387799; parent r_knee_servo_link -> r_thigh_link
- joint r_thigh_joint: origin xyz=0 0 0 rpy=0 0 -2.61799387799 -> xyz=0.02 0 -0.006 rpy=0 0 -2.61799387799; parent r_thigh_servo_link -> r_hip_link

Commit message: Fix shoulder joint/link

File: 2020/urdf/darwin.urdf (robot description, URDF)
Before this commit: robot darwin, 19 links, 18 joints
Joints:
- joint l_biceps_joint: origin xyz=0 0 0 rpy=-2.61799387799 0 0 -> xyz=0 0.018 -0.012 rpy=-2.61799387799 0 0
- joint l_shoulder_joint: axis 0 0 1 -> 0 1 0; origin xyz=-0.014 0.057 0.03 rpy=0 0 -2.61799387799 -> xyz=-0.014 0.039 0.042 rpy=0 -2.61799387799 0
- joint r_biceps_joint: origin xyz=0 0 0 rpy=-2.61799387799 0 0 -> xyz=0 -0.018 -0.012 rpy=-2.61799387799 0 0
- joint r_shoulder_joint: axis 0 0 1 -> 0 1 0; origin xyz=-0.014 -0.057 0.03 rpy=0 0 -2.61799387799 -> xyz=-0.014 -0.039 0.042 rpy=0 -2.61799387799 0

Commit message: Fix legs

File: 2020/urdf/darwin.urdf (robot description, URDF)
Before this commit: robot darwin, 19 links, 18 joints
Joints:
- joint l_ankle_joint: axis 0 0 1 -> 0 1 0; origin xyz=0 0 -0.042 rpy=0 0 -2.61799387799 -> xyz=0 0 -0.042 rpy=0 -2.61799387799 0
- joint l_elbow_joint: axis 0 0 1 -> 1 0 0; origin xyz=0 0 -0.044 rpy=0 0 -2.61799387799 -> xyz=0 0 -0.044 rpy=-2.61799387799 0 0
- joint l_foot_joint: axis 0 0 1 -> 1 0 0; origin xyz=-0.033 0 0 rpy=0 0 -2.61799387799 -> xyz=-0.033 0 0 rpy=-2.61799387799 0 0
- joint l_hip_joint: axis 0 0 1 -> 1 0 0; origin xyz=-0.024 0.024 -0.03 rpy=0 0 -2.61799387799 -> xyz=-0.024 0.024 -0.03 rpy=-2.61799387799 0 0
- joint l_knee_joint: axis 0 0 1 -> 0 1 0; origin xyz=0 0 -0.046 rpy=0 0 -2.61799387799 -> xyz=0 0 -0.046 rpy=0 -2.61799387799 0
- joint l_thigh_joint: axis 0 0 1 -> 0 1 0; origin xyz=0.02 0 -0.006 rpy=0 0 -2.61799387799 -> xyz=0.02 0 -0.006 rpy=0 -2.61799387799 0
- joint r_ankle_joint: axis 0 0 1 -> 0 1 0; origin xyz=0 0 -0.042 rpy=0 0 -2.61799387799 -> xyz=0 0 -0.042 rpy=0 -2.61799387799 0
- joint r_elbow_joint: axis 0 0 1 -> 1 0 0; origin xyz=0 0 -0.044 rpy=0 0 -2.61799387799 -> xyz=0 0 -0.044 rpy=-2.61799387799 0 0
- joint r_foot_joint: axis 0 0 1 -> 1 0 0; origin xyz=-0.033 0 0 rpy=0 0 -2.61799387799 -> xyz=-0.033 0 0 rpy=-2.61799387799 0 0
- joint r_hip_joint: axis 0 0 1 -> 1 0 0; origin xyz=-0.024 -0.024 -0.03 rpy=0 0 -2.61799387799 -> xyz=-0.024 -0.024 -0.03 rpy=-2.61799387799 0 0
- joint r_knee_joint: axis 0 0 1 -> 0 1 0; origin xyz=0 0 -0.046 rpy=0 0 -2.61799387799 -> xyz=0 0 -0.046 rpy=0 -2.61799387799 0
- joint r_thigh_joint: axis 0 0 1 -> 0 1 0; origin xyz=0.02 0 -0.006 rpy=0 0 -2.61799387799 -> xyz=0.02 0 -0.006 rpy=0 -2.61799387799 0

Commit message: Fix neck/head

File: 2020/urdf/darwin.urdf (robot description, URDF)
Before this commit: robot darwin, 19 links, 18 joints
Joints:
- joint neck_joint: origin xyz=0 0 0 rpy=0 0 -2.61799387799 -> xyz=-0.009 0 0.063 rpy=0 0 -2.61799387799
